File: defmon.brd (EAGLE design)
At the start: 50.8 x 48.1 mm, 18 parts, among them IC2 MEGA8-P, Q1 20MHz, X1 MAB5SH, X2 1503_09

Commit message: added the firmware
Parts:
- R1, R2: value 1k -> 220
Changed lines of the file:
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@@
 <setting verticaltext="up"/>
 </settings>
-<grid distance="0.05" unitdist="inch" unit="mm" style="lines" multiple="1" display="no" altdistance="0.025" altunitdist="inch" altunit="mm"/>
+<grid distance="0.05" unitdist="inch" unit="mil" style="lines" multiple="1" display="no" altdistance="0.025" altunitdist="inch" altunit="mil"/>
 <layers>
 <layer number="1" name="Top" color="4" fill="1" visible="yes" active="yes"/>
@@
 <attribute name="OC_FARNELL" value="unknown" x="12.7" y="27.94" size="1.778" layer="27" rot="R270" display="off"/>
 </element>
-<element name="R1" library="rcl" package="0204/7" value="1k" x="30.48" y="30.48" rot="R90"/>
+<element name="R1" library="rcl" package="0204/7" value="220" x="30.48" y="30.48" rot="R90"/>
 <element name="C3" library="rcl" package="C025-025X050" value="100nf" x="25.4" y="22.86" rot="R270"/>
 <element name="LED1" library="led" package="LED3MM" value="" x="29.21" y="19.05" rot="R90"/>
@@
 <element name="U$1" library="connector" package="GB" value="GB" x="48.768" y="0.762"/>
 <element name="U$2" library="connector" package="C64U" value="C64U" x="3.5" y="45.72" rot="R180"/>
-<element name="R2" library="rcl" package="0204/7" value="1k" x="33.02" y="30.48" rot="R90"/>
+<element name="R2" library="rcl" package="0204/7" value="220" x="33.02" y="30.48" rot="R90"/>
 <element name="LED2" library="led" package="LED3MM" value="" x="34.29" y="19.05" rot="R90"/>
 <element name="R3" library="rcl" package="0204/7" value="220" x="27.94" y="30.48" rot="R270"/>
@@
 </signal>
 <signal name="PE">
+<contactref element="X1" pad="PE"/>
 <contactref element="X1" pad="PE@"/>
-<contactref element="X1" pad="PE"/>
 <wire x1="48.26" y1="34.29" x2="48.26" y2="39.37" width="0" layer="19" extent="1-1"/>
 </signal>
@@
 <wire x1="34.29" y1="20.32" x2="33.02" y2="21.59" width="0.254" layer="16"/>
 <wire x1="33.02" y1="21.59" x2="33.02" y2="26.67" width="0.254" layer="16"/>
-</signal>
-<signal name="N$3">
-<contactref element="X1" pad="4"/>
-<contactref element="R3" pad="1"/>
-<wire x1="35.56" y1="41.91" x2="32.51905" y2="41.91" width="0.254" layer="16"/>
-<wire x1="32.51905" y1="41.91" x2="27.94" y2="37.33095" width="0.254" layer="16"/>
-<wire x1="27.94" y1="37.33095" x2="27.94" y2="34.29" width="0.254" layer="16"/>
 </signal>
 <signal name="N$4">
@@
 <wire x1="7.62" y1="6.02" x2="7.62" y2="6.35" width="0.6096" layer="1"/>
 </signal>
-<signal name="N$7">
-<contactref element="X1" pad="5"/>
-<contactref element="IC2" pad="3"/>
-<wire x1="35.56" y1="31.75" x2="28.46605" y2="31.75" width="0.254" layer="16"/>
-<wire x1="28.46605" y1="31.75" x2="25.4" y2="34.81605" width="0.254" layer="16"/>
-<wire x1="25.4" y1="34.81605" x2="25.4" y2="36.30395" width="0.254" layer="16"/>
-<wire x1="25.4" y1="36.30395" x2="23.60395" y2="38.1" width="0.254" layer="16"/>
-<wire x1="23.60395" y1="38.1" x2="15.24" y2="38.1" width="0.254" layer="16"/>
-<wire x1="15.24" y1="38.1" x2="13.97" y2="39.37" width="0.254" layer="16"/>
-</signal>
 <signal name="TRIG1">
 <contactref element="IC2" pad="23"/>
@@
 <wire x1="13.97" y1="44.45" x2="10.16" y2="44.45" width="0.254" layer="16"/>
 </signal>
+<signal name="N$13">
+<contactref element="IC2" pad="3"/>
+<contactref element="X1" pad="5"/>
+<wire x1="35.56" y1="31.75" x2="28.23980625" y2="31.75" width="0.254" layer="16"/>
+<wire x1="28.23980625" y1="31.75" x2="25.4" y2="34.58980625" width="0.254" layer="16"/>
+<wire x1="25.4" y1="34.58980625" x2="25.4" y2="36.30395" width="0.254" layer="16"/>
+<wire x1="25.4" y1="36.30395" x2="23.60395" y2="38.1" width="0.254" layer="16"/>
+<wire x1="23.60395" y1="38.1" x2="15.24" y2="38.1" width="0.254" layer="16"/>
+<wire x1="15.24" y1="38.1" x2="13.97" y2="39.37" width="0.254" layer="16"/>
+</signal>
+<signal name="N$3">
+<contactref element="X1" pad="4"/>
+<contactref element="R3" pad="1"/>
+<wire x1="35.56" y1="41.91" x2="33.328153125" y2="41.91" width="0.254" layer="16"/>
+<wire x1="33.328153125" y1="41.91" x2="27.94" y2="36.521846875" width="0.254" layer="16"/>
+<wire x1="27.94" y1="36.521846875" x2="27.94" y2="34.29" width="0.254" layer="16"/>
+</signal>
 </signals>
