File: defmon.sch (EAGLE design)
At the start: 18 parts, among them IC2 MEGA8-P, Q1 20MHz, X1 MAB5SH, X2 1503_09

Commit message: added the firmware
Parts:
- R1, R2: value 1k -> 220
Other:
- moved on the sheet: R3
Changed lines of the file:
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@@
 <part name="P+13" library="supply1" deviceset="VCC" device=""/>
 <part name="GND20" library="supply1" deviceset="GND" device=""/>
-<part name="R1" library="rcl" deviceset="R-US_" device="0204/7" value="1k"/>
+<part name="R1" library="rcl" deviceset="R-US_" device="0204/7" value="220"/>
 <part name="C3" library="rcl" deviceset="C-US" device="025-025X050" value="100nf"/>
 <part name="GND5" library="supply1" deviceset="GND" device=""/>
@@
 <part name="P+1" library="supply1" deviceset="VCC" device=""/>
 <part name="GND2" library="supply1" deviceset="GND" device=""/>
-<part name="R2" library="rcl" deviceset="R-US_" device="0204/7" value="1k"/>
+<part name="R2" library="rcl" deviceset="R-US_" device="0204/7" value="220"/>
 <part name="LED2" library="led" deviceset="LED" device="3MM"/>
 <part name="R3" library="rcl" deviceset="R-US_" device="0204/7" value="220"/>
@@
 <instance part="R2" gate="G$1" x="154.94" y="172.72"/>
 <instance part="LED2" gate="G$1" x="142.24" y="172.72" rot="R90"/>
-<instance part="R3" gate="G$1" x="193.04" y="228.6"/>
+<instance part="R3" gate="G$1" x="198.12" y="228.6"/>
 <instance part="GND3" gate="1" x="185.42" y="220.98"/>
-<instance part="P+2" gate="VCC" x="200.66" y="233.68"/>
+<instance part="P+2" gate="VCC" x="205.74" y="236.22"/>
 <instance part="GND4" gate="1" x="165.1" y="177.8"/>
 <instance part="P+3" gate="VCC" x="259.08" y="238.76"/>
@@
 <pinref part="R3" gate="G$1" pin="2"/>
 <pinref part="P+2" gate="VCC" pin="VCC"/>
-<wire x1="198.12" y1="228.6" x2="200.66" y2="228.6" width="0.1524" layer="91"/>
-<wire x1="200.66" y1="228.6" x2="200.66" y2="231.14" width="0.1524" layer="91"/>
+<wire x1="203.2" y1="228.6" x2="205.74" y2="228.6" width="0.1524" layer="91"/>
+<wire x1="205.74" y1="228.6" x2="205.74" y2="233.68" width="0.1524" layer="91"/>
 </segment>
 <segment>
@@
 <pinref part="R2" gate="G$1" pin="1"/>
 <wire x1="147.32" y1="172.72" x2="149.86" y2="172.72" width="0.1524" layer="91"/>
-</segment>
-</net>
-<net name="N$3" class="0">
-<segment>
-<pinref part="X1" gate="G$1" pin="4"/>
-<pinref part="R3" gate="G$1" pin="1"/>
-<wire x1="180.34" y1="228.6" x2="187.96" y2="228.6" width="0.1524" layer="91"/>
 </segment>
 </net>
@@
 <wire x1="134.62" y1="185.42" x2="137.16" y2="185.42" width="0.1524" layer="91"/>
 <label x="134.62" y="185.42" size="1.778" layer="95"/>
-</segment>
-</net>
-<net name="N$7" class="0">
-<segment>
-<pinref part="X1" gate="G$1" pin="5"/>
-<wire x1="154.94" y1="228.6" x2="152.4" y2="228.6" width="0.1524" layer="91"/>
-<pinref part="IC2" gate="G$1" pin="PD1(TXD)"/>
-<wire x1="134.62" y1="205.74" x2="152.4" y2="205.74" width="0.1524" layer="91"/>
-<wire x1="152.4" y1="205.74" x2="152.4" y2="228.6" width="0.1524" layer="91"/>
 </segment>
 </net>
@@
 </segment>
 </net>
+<net name="N$13" class="0">
+<segment>
+<pinref part="IC2" gate="G$1" pin="PD1(TXD)"/>
+<wire x1="134.62" y1="205.74" x2="152.4" y2="205.74" width="0.1524" layer="91"/>
+<pinref part="X1" gate="G$1" pin="5"/>
+<wire x1="154.94" y1="228.6" x2="152.4" y2="228.6" width="0.1524" layer="91"/>
+<wire x1="152.4" y1="205.74" x2="152.4" y2="228.6" width="0.1524" layer="91"/>
+</segment>
+</net>
+<net name="N$3" class="0">
+<segment>
+<pinref part="X1" gate="G$1" pin="4"/>
+<wire x1="180.34" y1="228.6" x2="193.04" y2="228.6" width="0.1524" layer="91"/>
+<pinref part="R3" gate="G$1" pin="1"/>
+</segment>
+</net>
